Commit message: フォイル階層を整理

File: urdf/mycobot_280_m5/mycobot_280_m5.urdf (robot description, URDF)
Before this commit: robot firefighter, 8 links, 7 joints
Links:
- link g_base: geometry collision mesh filename=package://three_d_mouse_leader/meshes/mycobot_280_m5/G_base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; visual mesh filename=package://three_d_mouse_leader/meshes/mycobot_280_m5/G_base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
- link joint1: geometry collision mesh filename=package://three_d_mouse_leader/meshes/mycobot_280_m5/joint1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; visual mesh filename=package://three_d_mouse_leader/meshes/mycobot_280_m5/joint1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
- link joint2: geometry collision mesh filename=package://three_d_mouse_leader/meshes/mycobot_280_m5/joint2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; visual mesh filename=package://three_d_mouse_leader/meshes/mycobot_280_m5/joint2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
- link joint3: geometry collision mesh filename=package://three_d_mouse_leader/meshes/mycobot_280_m5/joint3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; visual mesh filename=package://three_d_mouse_leader/meshes/mycobot_280_m5/joint3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
- link joint4: geometry collision mesh filename=package://three_d_mouse_leader/meshes/mycobot_280_m5/joint4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; visual mesh filename=package://three_d_mouse_leader/meshes/mycobot_280_m5/joint4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
- link joint5: geometry collision mesh filename=package://three_d_mouse_leader/meshes/mycobot_280_m5/joint5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; visual mesh filename=package://three_d_mouse_leader/meshes/mycobot_280_m5/joint5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
- link joint6: geometry collision mesh filename=package://three_d_mouse_leader/meshes/mycobot_280_m5/joint6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; visual mesh filename=package://three_d_mouse_leader/meshes/mycobot_280_m5/joint6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
- link joint6_flange: geometry collision mesh filename=package://three_d_mouse_leader/meshes/mycobot_280_m5/joint7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; visual mesh filename=package://three_d_mouse_leader/meshes/mycobot_280_m5/joint7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

File: urdf/mycobot_280_m5/mycobot_280_m5_adaptive_gripper.urdf (robot description, URDF)
Before this commit: robot firefighter, 15 links, 14 joints
Links:
- link g_base: geometry collision mesh filename=package://three_d_mouse_leader/meshes/mycobot_280_m5/G_base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; visual mesh filename=package://three_d_mouse_leader/meshes/mycobot_280_m5/G_base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
- link joint1: geometry collision mesh filename=package://three_d_mouse_leader/meshes/mycobot_280_m5/joint1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; visual mesh filename=package://three_d_mouse_leader/meshes/mycobot_280_m5/joint1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
- link joint2: geometry collision mesh filename=package://three_d_mouse_leader/meshes/mycobot_280_m5/joint2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; visual mesh filename=package://three_d_mouse_leader/meshes/mycobot_280_m5/joint2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
- link joint3: geometry collision mesh filename=package://three_d_mouse_leader/meshes/mycobot_280_m5/joint3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; visual mesh filename=package://three_d_mouse_leader/meshes/mycobot_280_m5/joint3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
- link joint4: geometry collision mesh filename=package://three_d_mouse_leader/meshes/mycobot_280_m5/joint4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; visual mesh filename=package://three_d_mouse_leader/meshes/mycobot_280_m5/joint4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
- link joint5: geometry collision mesh filename=package://three_d_mouse_leader/meshes/mycobot_280_m5/joint5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; visual mesh filename=package://three_d_mouse_leader/meshes/mycobot_280_m5/joint5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
- link joint6: geometry collision mesh filename=package://three_d_mouse_leader/meshes/mycobot_280_m5/joint6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; visual mesh filename=package://three_d_mouse_leader/meshes/mycobot_280_m5/joint6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
- link joint6_flange: geometry collision mesh filename=package://three_d_mouse_leader/meshes/mycobot_280_m5/joint7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; visual mesh filename=package://three_d_mouse_leader/meshes/mycobot_280_m5/joint7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

File: urdf/mycobot_280_m5/mycobot_280_m5_with_camera_flange.urdf (robot description, URDF)
Before this commit: robot firefighter, 9 links, 8 joints
Links:
- link camera_flange: geometry collision mesh filename=package://three_d_mouse_leader/meshes/mycobot_280_m5/camera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; visual mesh filename=package://three_d_mouse_leader/meshes/mycobot_280_m5/camera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
- link g_base: geometry collision mesh filename=package://three_d_mouse_leader/meshes/mycobot_280_m5/G_base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; visual mesh filename=package://three_d_mouse_leader/meshes/mycobot_280_m5/G_base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
- link joint1: geometry collision mesh filename=package://three_d_mouse_leader/meshes/mycobot_280_m5/joint1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; visual mesh filename=package://three_d_mouse_leader/meshes/mycobot_280_m5/joint1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
- link joint2: geometry collision mesh filename=package://three_d_mouse_leader/meshes/mycobot_280_m5/joint2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; visual mesh filename=package://three_d_mouse_leader/meshes/mycobot_280_m5/joint2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
- link joint3: geometry collision mesh filename=package://three_d_mouse_leader/meshes/mycobot_280_m5/joint3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; visual mesh filename=package://three_d_mouse_leader/meshes/mycobot_280_m5/joint3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
- link joint4: geometry collision mesh filename=package://three_d_mouse_leader/meshes/mycobot_280_m5/joint4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; visual mesh filename=package://three_d_mouse_leader/meshes/mycobot_280_m5/joint4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
- link joint5: geometry collision mesh filename=package://three_d_mouse_leader/meshes/mycobot_280_m5/joint5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; visual mesh filename=package://three_d_mouse_leader/meshes/mycobot_280_m5/joint5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
- link joint6: geometry collision mesh filename=package://three_d_mouse_leader/meshes/mycobot_280_m5/joint6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; visual mesh filename=package://three_d_mouse_leader/meshes/mycobot_280_m5/joint6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
- link joint6_flange: geometry collision mesh filename=package://three_d_mouse_leader/meshes/mycobot_280_m5/joint7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; visual mesh filename=package://three_d_mouse_leader/meshes/mycobot_280_m5/joint7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

File: urdf/mycobot_280_m5/mycobot_280_m5_with_camera_flange_pump.urdf (robot description, URDF)
Before this commit: robot firefighter, 11 links, 10 joints
Links:
- link camera_flange: geometry collision mesh filename=package://three_d_mouse_leader/meshes/mycobot_280_m5/camera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; visual mesh filename=package://three_d_mouse_leader/meshes/mycobot_280_m5/camera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
- link g_base: geometry collision mesh filename=package://three_d_mouse_leader/meshes/mycobot_280_m5/G_base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; visual mesh filename=package://three_d_mouse_leader/meshes/mycobot_280_m5/G_base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
- link joint1: geometry collision mesh filename=package://three_d_mouse_leader/meshes/mycobot_280_m5/joint1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; visual mesh filename=package://three_d_mouse_leader/meshes/mycobot_280_m5/joint1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
- link joint2: geometry collision mesh filename=package://three_d_mouse_leader/meshes/mycobot_280_m5/joint2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; visual mesh filename=package://three_d_mouse_leader/meshes/mycobot_280_m5/joint2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
- link joint3: geometry collision mesh filename=package://three_d_mouse_leader/meshes/mycobot_280_m5/joint3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; visual mesh filename=package://three_d_mouse_leader/meshes/mycobot_280_m5/joint3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
- link joint4: geometry collision mesh filename=package://three_d_mouse_leader/meshes/mycobot_280_m5/joint4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; visual mesh filename=package://three_d_mouse_leader/meshes/mycobot_280_m5/joint4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
- link joint5: geometry collision mesh filename=package://three_d_mouse_leader/meshes/mycobot_280_m5/joint5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; visual mesh filename=package://three_d_mouse_leader/meshes/mycobot_280_m5/joint5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
- link joint6: geometry collision mesh filename=package://three_d_mouse_leader/meshes/mycobot_280_m5/joint6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; visual mesh filename=package://three_d_mouse_leader/meshes/mycobot_280_m5/joint6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
- link joint6_flange: geometry collision mesh filename=package://three_d_mouse_leader/meshes/mycobot_280_m5/joint7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; visual mesh filename=package://three_d_mouse_leader/meshes/mycobot_280_m5/joint7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
- link pump_box: geometry collision mesh filename=package://three_d_mouse_leader/meshes/mycobot_280_m5/pump_b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; visual mesh filename=package://three_d_mouse_leader/meshes/mycobot_280_m5/pump_b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
- link pump_head: geometry collision mesh filename=package://three_d_mouse_leader/meshes/mycobot_280_m5/pump_h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; visual mesh filename=package://three_d_mouse_leader/meshes/mycobot_280_m5/pump_h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

File: urdf/mycobot_280_m5/mycobot_280_m5_with_pump.urdf (robot description, URDF)
Before this commit: robot firefighter, 10 links, 9 joints
Links:
- link g_base: geometry collision mesh filename=package://three_d_mouse_leader/meshes/mycobot_280_m5/G_base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; visual mesh filename=package://three_d_mouse_leader/meshes/mycobot_280_m5/G_base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
- link joint1: geometry collision mesh filename=package://three_d_mouse_leader/meshes/mycobot_280_m5/joint1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; visual mesh filename=package://three_d_mouse_leader/meshes/mycobot_280_m5/joint1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
- link joint2: geometry collision mesh filename=package://three_d_mouse_leader/meshes/mycobot_280_m5/joint2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; visual mesh filename=package://three_d_mouse_leader/meshes/mycobot_280_m5/joint2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
- link joint3: geometry collision mesh filename=package://three_d_mouse_leader/meshes/mycobot_280_m5/joint3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; visual mesh filename=package://three_d_mouse_leader/meshes/mycobot_280_m5/joint3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
- link joint4: geometry collision mesh filename=package://three_d_mouse_leader/meshes/mycobot_280_m5/joint4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; visual mesh filename=package://three_d_mouse_leader/meshes/mycobot_280_m5/joint4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
- link joint5: geometry collision mesh filename=package://three_d_mouse_leader/meshes/mycobot_280_m5/joint5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; visual mesh filename=package://three_d_mouse_leader/meshes/mycobot_280_m5/joint5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
- link joint6: geometry collision mesh filename=package://three_d_mouse_leader/meshes/mycobot_280_m5/joint6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; visual mesh filename=package://three_d_mouse_leader/meshes/mycobot_280_m5/joint6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
- link joint6_flange: geometry collision mesh filename=package://three_d_mouse_leader/meshes/mycobot_280_m5/joint7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; visual mesh filename=package://three_d_mouse_leader/meshes/mycobot_280_m5/joint7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
- link pump_box: geometry collision mesh filename=package://three_d_mouse_leader/meshes/mycobot_280_m5/pump_b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; visual mesh filename=package://three_d_mouse_leader/meshes/mycobot_280_m5/pump_b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
- link pump_head: geometry collision mesh filename=package://three_d_mouse_leader/meshes/mycobot_280_m5/pump_h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; visual mesh filename=package://three_d_mouse_leader/meshes/mycobot_280_m5/pump_h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

File: urdf/mycobot_280_m5/mycobot_with_vision.urdf (robot description, URDF)
Before this commit: robot mycobot_ai, 8 links, 7 joints
Links:
- link env: geometry visual mesh filename=package://three_d_mouse_leader/meshes/mycobot_280_m5/suit_e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
- link joint1: geometry collision mesh filename=package://three_d_mouse_leader/meshes/mycobot_280_m5/joint1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; visual mesh filename=package://three_d_mouse_leader/meshes/mycobot_280_m5/joint1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
- link joint2: geometry collision mesh filename=package://three_d_mouse_leader/meshes/mycobot_280_m5/joint2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; visual mesh filename=package://three_d_mouse_leader/meshes/mycobot_280_m5/joint2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
- link joint3: geometry collision mesh filename=package://three_d_mouse_leader/meshes/mycobot_280_m5/joint3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; visual mesh filename=package://three_d_mouse_leader/meshes/mycobot_280_m5/joint3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
- link joint4: geometry collision mesh filename=package://three_d_mouse_leader/meshes/mycobot_280_m5/joint4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; visual mesh filename=package://three_d_mouse_leader/meshes/mycobot_280_m5/joint4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
- link joint5: geometry collision mesh filename=package://three_d_mouse_leader/meshes/mycobot_280_m5/joint5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; visual mesh filename=package://three_d_mouse_leader/meshes/mycobot_280_m5/joint5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
- link joint6: geometry collision mesh filename=package://three_d_mouse_leader/meshes/mycobot_280_m5/joint6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; visual mesh filename=package://three_d_mouse_leader/meshes/mycobot_280_m5/joint6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
- link joint6_flange: geometry collision mesh filename=package://three_d_mouse_leader/meshes/mycobot_280_m5/joint7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; visual mesh filename=package://three_d_mouse_leader/meshes/mycobot_280_m5/joint7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

File: urdf/mycobot_280_m5/mycobot_with_vision_copy.urdf (robot description, URDF)
Before this commit: robot mycobot_ai, 1 links, 1 joints
Links:
- link env: geometry visual mesh filename=package://three_d_mouse_leader/meshes/mycobot_280_m5/suit_e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
