Commit message: グリッパ付きURDFの有効化

File: urdf/mycobot_280_m5/mycobot_280_m5_adaptive_gripper.urdf (robot description, URDF)
Before this commit: robot firefighter, 15 links, 14 joints
Links:
- link gripper_base: geometry collision mesh filename=package://three_d_mouse_leader/meshes/mycobot_280_m5/adapti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; visual mesh filename=package://three_d_mouse_leader/meshes/mycobot_280_m5/adapti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
- link gripper_left1: geometry collision mesh filename=package://three_d_mouse_leader/meshes/mycobot_280_m5/adapti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; visual mesh filename=package://three_d_mouse_leader/meshes/mycobot_280_m5/adapti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
- link gripper_left2: geometry collision mesh filename=package://three_d_mouse_leader/meshes/mycobot_280_m5/adapti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; visual mesh filename=package://three_d_mouse_leader/meshes/mycobot_280_m5/adapti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
- link gripper_left3: geometry collision mesh filename=package://three_d_mouse_leader/meshes/mycobot_280_m5/adapti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; visual mesh filename=package://three_d_mouse_leader/meshes/mycobot_280_m5/adapti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
- link gripper_right1: geometry collision mesh filename=package://three_d_mouse_leader/meshes/mycobot_280_m5/adapti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; visual mesh filename=package://three_d_mouse_leader/meshes/mycobot_280_m5/adapti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
- link gripper_right2: geometry collision mesh filename=package://three_d_mouse_leader/meshes/mycobot_280_m5/adapti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; visual mesh filename=package://three_d_mouse_leader/meshes/mycobot_280_m5/adapti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
- link gripper_right3: geometry collision mesh filename=package://three_d_mouse_leader/meshes/mycobot_280_m5/adapti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; visual mesh filename=package://three_d_mouse_leader/meshes/mycobot_280_m5/adapti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
